File: hw/breakout/breakout.sch (KiCad schematic (older format))
At the start: 42 parts, among them J1 Rain, J10 SPI_CS, J11 Uart, J12 GPS, J13 RX_SEL, J2 Wind, J3 ARM-SWD, J4 PWR_IN, J5 PWR, J6 GPIO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

Commit message: Finished breakout v0.0.1
Parts:
- removed TP1, TP2: TEST, symbol TEST
- added C5, C6: 1uF, Capacitors_SMD:C_0603, symbol C_Small
- C1, C2, C3, C4: footprint (none) -> Capacitors_SMD:C_0603
- D1, D2, D3, D4: footprint (none) -> LEDs:LED_0603
- J1, J2: footprint (none) -> alvarop:RJ11
- J10, J5, J6, J8, J9: footprint (none) -> Pin_Headers:Pin_Header_Straight_1x04_Pitch2.54mm
- J11: footprint (none) -> Pin_Headers:Pin_Header_Straight_1x06_Pitch2.54mm
- J12, J13, J7: footprint (none) -> Pin_Headers:Pin_Header_Straight_1x03_Pitch2.54mm
- J3: footprint (none) -> alvarop:ARM_SWD_SMD
- J4: footprint (none) -> Pin_Headers:Pin_Header_Straight_1x02_Pitch2.54mm
- L1: footprint (none) -> Resistors_SMD:R_0603; DKPN (none) -> 587-1547-1-ND; MPN (none) -> HK160815NJ-T
- L2: footprint (none) -> Resistors_SMD:R_0603; DKPN (none) -> 587-1714-1-ND; MPN (none) -> LBMF1608T100K
- R1, R10, R11, R12, R13, R2, R3, R4, R5, R6, R7, R8, R9: footprint (none) -> Resistors_SMD:R_0603
- U1: footprint (none) -> alvarop:SOT-23(M5)
- U2: footprint (none) -> alvarop:SHT3x
- U3: footprint (none) -> alvarop:MDBT42Q
- Y1: footprint (none) -> alvarop:FC-135
Connections:
- net +3V3: now also J7.1 (Pin_1), C6.1; no longer J7.3 (Pin_3)
- net GND: now also C5.2, C6.2
- net LIGHT: now also J7.3 (Pin_3); no longer J7.1 (Pin_1)
- net SCL: now also U3.3 (P0.26); no longer U3.4 (P0.27)
- net SDA: now also U3.4 (P0.27); no longer U3.3 (P0.26)
- net V_IN: now also C5.1
- net RAIN2: no longer names the net of J1.2
- net RAIN5: no longer names the net of J1.5
- no-connect marks 20 -> 22

Commit message: Added MPNs to breakout.sch
Parts:
- C1, C2: DKPN (none) -> 1276-2175-1-ND; MPN (none) -> CL10C120FB8NNNC
- C3: DKPN (none) -> 490-3896-1-ND; MPN (none) -> GRM188R60J106ME47D
- C4, C5, C6: DKPN (none) -> 1276-1867-1-ND; MPN (none) -> CL10A105MQ8NNNC
- D1, D2, D3, D4: DKPN (none) -> 160-1183-1-ND; MPN (none) -> LTST-C190GKT
- J3: DKPN (none) -> 609-3695-1-ND; MPN (none) -> 20021121-00010C4LF
- R1, R10, R11, R2, R3, R4, R5, R6, R8, R9: DKPN (none) -> 311-1.0KGRCT-ND; MPN (none) -> RC0603JR-071KL
- R12, R13, R7: DKPN (none) -> 311-4.7KGRCT-ND; MPN (none) -> RC0603JR-074K7L
- U1: DKPN (none) -> 576-4764-1-ND; MPN (none) -> MIC5504-3.3YM5-TR
- U2: DKPN (none) -> 1649-1066-1-ND; MPN (none) -> SHT31-DIS-F2.5KS
Changed lines of the file:
@@
 F 2 "Capacitors_SMD:C_0603" H 3500 1350 50  0001 C CNN
 F 3 "" H 3500 1350 50  0001 C CNN
+F 4 "CL10C120FB8NNNC" H 3500 1350 60  0001 C CNN "MPN"
+F 5 "1276-2175-1-ND" H 3500 1350 60  0001 C CNN "DKPN"
 	1    3500 1350
 	-1   0    0    1
@@
 F 2 "Capacitors_SMD:C_0603" H 3900 1350 50  0001 C CNN
 F 3 "" H 3900 1350 50  0001 C CNN
+F 4 "CL10C120FB8NNNC" H 3900 1350 60  0001 C CNN "MPN"
+F 5 "1276-2175-1-ND" H 3900 1350 60  0001 C CNN "DKPN"
 	1    3900 1350
 	-1   0    0    1
@@
 F 2 "Resistors_SMD:R_0603" H 1700 5400 50  0001 C CNN
 F 3 "" H 1700 5400 50  0001 C CNN
+F 4 "RC0603JR-071KL" V 2000 3350 60  0001 C CNN "MPN"
+F 5 "311-1.0KGRCT-ND" V 2000 3350 60  0001 C CNN "DKPN"
 	1    1700 5400
 	1    0    0    -1
@@
 F 2 "Resistors_SMD:R_0603" H 1550 5400 50  0001 C CNN
 F 3 "" H 1550 5400 50  0001 C CNN
+F 4 "RC0603JR-071KL" V 2000 3350 60  0001 C CNN "MPN"
+F 5 "311-1.0KGRCT-ND" V 2000 3350 60  0001 C CNN "DKPN"
 	1    1550 5400
 	1    0    0    -1
@@
 F 2 "Resistors_SMD:R_0603" H 1700 4900 50  0001 C CNN
 F 3 "" H 1700 4900 50  0001 C CNN
+F 4 "RC0603JR-071KL" V 2000 3350 60  0001 C CNN "MPN"
+F 5 "311-1.0KGRCT-ND" V 2000 3350 60  0001 C CNN "DKPN"
 	1    1700 4900
 	0    -1   -1   0
@@
 F 2 "Resistors_SMD:R_0603" H 1700 5000 50  0001 C CNN
 F 3 "" H 1700 5000 50  0001 C CNN
+F 4 "RC0603JR-071KL" V 2000 3350 60  0001 C CNN "MPN"
+F 5 "311-1.0KGRCT-ND" V 2000 3350 60  0001 C CNN "DKPN"
 	1    1700 5000
 	0    -1   -1   0
@@
 F 2 "Resistors_SMD:R_0603" H 2050 4700 50  0001 C CNN
 F 3 "" H 2050 4700 50  0001 C CNN
+F 4 "RC0603JR-074K7L" V 2050 4700 60  0001 C CNN "MPN"
+F 5 "311-4.7KGRCT-ND" V 2050 4700 60  0001 C CNN "DKPN"
 	1    2050 4700
 	1    0    0    -1
@@
 F 2 "Resistors_SMD:R_0603" H 1900 3650 50  0001 C CNN
 F 3 "" H 1900 3650 50  0001 C CNN
+F 4 "RC0603JR-071KL" V 2000 3350 60  0001 C CNN "MPN"
+F 5 "311-1.0KGRCT-ND" V 2000 3350 60  0001 C CNN "DKPN"
 	1    1900 3650
 	1    0    0    -1
@@
 F 2 "Resistors_SMD:R_0603" H 2000 3350 50  0001 C CNN
 F 3 "" H 2000 3350 50  0001 C CNN
+F 4 "RC0603JR-071KL" V 2000 3350 60  0001 C CNN "MPN"
+F 5 "311-1.0KGRCT-ND" V 2000 3350 60  0001 C CNN "DKPN"
 	1    2000 3350
 	0    -1   -1   0
@@
 F 2 "alvarop:SHT3x" H 1800 6550 60  0001 C CNN
 F 3 "" H 1800 6550 60  0000 C CNN
+F 4 "SHT31-DIS-F2.5KS" H 2050 6550 60  0001 C CNN "MPN"
+F 5 "1649-1066-1-ND" H 2050 6550 60  0001 C CNN "DKPN"
 	1    2050 6550
 	1    0    0    -1
@@
 F 2 "Resistors_SMD:R_0603" H 8600 1350 50  0001 C CNN
 F 3 "" H 8600 1350 50  0001 C CNN
+F 4 "RC0603JR-074K7L" V 8600 1350 60  0001 C CNN "MPN"
+F 5 "311-4.7KGRCT-ND" V 8600 1350 60  0001 C CNN "DKPN"
 	1    8600 1350
 	1    0    0    -1
@@
 F 2 "Resistors_SMD:R_0603" H 8300 1350 50  0001 C CNN
 F 3 "" H 8300 1350 50  0001 C CNN
+F 4 "RC0603JR-074K7L" V 8300 1350 60  0001 C CNN "MPN"
+F 5 "311-4.7KGRCT-ND" V 8300 1350 60  0001 C CNN "DKPN"
 	1    8300 1350
 	1    0    0    -1
@@
 F 2 "alvarop:ARM_SWD_SMD" H 5050 7050 60  0001 C CNN
 F 3 "" H 5050 7050 60  0000 C CNN
+F 4 "20021121-00010C4LF" H 5350 7200 60  0001 C CNN "MPN"
+F 5 "609-3695-1-ND" H 5350 7200 60  0001 C CNN "DKPN"
 	1    5350 7200
 	1    0    0    -1
@@
 F 2 "Capacitors_SMD:C_0603" H 6550 1600 50  0001 C CNN
 F 3 "" H 6550 1600 50  0001 C CNN
+F 4 "CL10A105MQ8NNNC" H 6550 1600 60  0001 C CNN "MPN"
+F 5 "1276-1867-1-ND" H 6550 1600 60  0001 C CNN "DKPN"
 	1    6550 1600
 	1    0    0    -1
@@
 F 2 "alvarop:SOT-23(M5)" H 1950 1400 60  0001 C CNN
 F 3 "" H 1950 1400 60  0000 C CNN
+F 4 "MIC5504-3.3YM5-TR" H 1950 1400 60  0001 C CNN "MPN"
+F 5 "576-4764-1-ND" H 1950 1400 60  0001 C CNN "DKPN"
 	1    1950 1400
 	1    0    0    -1
@@
 F 2 "Capacitors_SMD:C_0603" H 5600 2100 50  0001 C CNN
 F 3 "" H 5600 2100 50  0001 C CNN
+F 4 "GRM188R60J106ME47D" H 5600 2100 60  0001 C CNN "MPN"
+F 5 "490-3896-1-ND" H 5600 2100 60  0001 C CNN "DKPN"
 	1    5600 2100
 	1    0    0    -1
@@
 F 2 "LEDs:LED_0603" H 3000 7100 50  0001 C CNN
 F 3 "" H 3000 7100 50  0001 C CNN
+F 4 "LTST-C190GKT" H 3000 7100 60  0001 C CNN "MPN"
+F 5 "160-1183-1-ND" H 3000 7100 60  0001 C CNN "DKPN"
 	1    3000 7100
 	0    -1   -1   0
@@
 F 2 "LEDs:LED_0603" H 3300 7100 50  0001 C CNN
 F 3 "" H 3300 7100 50  0001 C CNN
+F 4 "LTST-C190GKT" H 3300 7100 60  0001 C CNN "MPN"
+F 5 "160-1183-1-ND" H 3300 7100 60  0001 C CNN "DKPN"
 	1    3300 7100
 	0    -1   -1   0
@@
 F 2 "LEDs:LED_0603" H 3600 7100 50  0001 C CNN
 F 3 "" H 3600 7100 50  0001 C CNN
+F 4 "LTST-C190GKT" H 3600 7100 60  0001 C CNN "MPN"
+F 5 "160-1183-1-ND" H 3600 7100 60  0001 C CNN "DKPN"
 	1    3600 7100
 	0    -1   -1   0
@@
 F 2 "LEDs:LED_0603" H 3900 7100 50  0001 C CNN
 F 3 "" H 3900 7100 50  0001 C CNN
+F 4 "LTST-C190GKT" H 3900 7100 60  0001 C CNN "MPN"
+F 5 "160-1183-1-ND" H 3900 7100 60  0001 C CNN "DKPN"
 	1    3900 7100
 	0    -1   -1   0
@@
 F 2 "Resistors_SMD:R_0603" H 3000 6800 50  0001 C CNN
 F 3 "" H 3000 6800 50  0001 C CNN
+F 4 "RC0603JR-071KL" V 2000 3350 60  0001 C CNN "MPN"
+F 5 "311-1.0KGRCT-ND" V 2000 3350 60  0001 C CNN "DKPN"
 	1    3000 6800
 	1    0    0    -1
@@
 F 2 "Resistors_SMD:R_0603" H 3300 6800 50  0001 C CNN
 F 3 "" H 3300 6800 50  0001 C CNN
+F 4 "RC0603JR-071KL" V 2000 3350 60  0001 C CNN "MPN"
+F 5 "311-1.0KGRCT-ND" V 2000 3350 60  0001 C CNN "DKPN"
 	1    3300 6800
 	1    0    0    -1
@@
 F 2 "Resistors_SMD:R_0603" H 3600 6800 50  0001 C CNN
 F 3 "" H 3600 6800 50  0001 C CNN
+F 4 "RC0603JR-071KL" V 2000 3350 60  0001 C CNN "MPN"
+F 5 "311-1.0KGRCT-ND" V 2000 3350 60  0001 C CNN "DKPN"
 	1    3600 6800
 	1    0    0    -1
@@
 F 2 "Resistors_SMD:R_0603" H 3900 6800 50  0001 C CNN
 F 3 "" H 3900 6800 50  0001 C CNN
+F 4 "RC0603JR-071KL" V 2000 3350 60  0001 C CNN "MPN"
+F 5 "311-1.0KGRCT-ND" V 2000 3350 60  0001 C CNN "DKPN"
 	1    3900 6800
 	1    0    0    -1
@@
 F 2 "Capacitors_SMD:C_0603" H 2500 1400 50  0001 C CNN
 F 3 "" H 2500 1400 50  0001 C CNN
+F 4 "CL10A105MQ8NNNC" H 2500 1400 60  0001 C CNN "MPN"
+F 5 "1276-1867-1-ND" H 2500 1400 60  0001 C CNN "DKPN"
 	1    2500 1400
 	1    0    0    -1
@@
 F 2 "Capacitors_SMD:C_0603" H 1450 1400 50  0001 C CNN
 F 3 "" H 1450 1400 50  0001 C CNN
+F 4 "CL10A105MQ8NNNC" H 1450 1400 60  0001 C CNN "MPN"
+F 5 "1276-1867-1-ND" H 1450 1400 60  0001 C CNN "DKPN"
 	1    1450 1400
 	1    0    0    -1
